File: 6lowPan/bontor_mbed_lowpan_rev_f.sch (EAGLE design)
At the start: 170 parts, among them IC1 SIM900, IC2 74HC595D, IC3 74HC595D, IC4 ADE7758RW, IC5 74HC595D, J1 U.FL, U2 W5500, X1 NX2520SA

Commit message: update silkscreen and delete USB micro hole
Parts:
- removed SIM900-R4: 680R, rcl:R-EU_R0402
- removed STM-C12, STM-C9: 100nF, rcl:C-EUC0603
- added C25, LCD_C1: 100nF, rcl:C-EUC0603
- added C27: 100nF, rcl:C-EUC0402
- added C28: 4.7uF, rcl:C-EUC0603
- added R94: 680R, rcl:R-EU_R0603
- ESP: value ESP8266WI12 -> ESP
- S1: device SparkFun-Electromechanical:TAC_SWITCHSMD -> SparkFun-Electromechanical:TAC_SWITCHPTH
- renumbered ADE-C1 to C71, ADE-C2 to C72, ADE-C3 to C73, ADE-C4 to C74, ADE-C6 to C70, CC_C14 to C46, CC_C20 to C41, CC_C8 to C43, CC_CX1 to C44, CC_CX2 to C45, CC_DCOUP to C40, ETH-C1 to C36, ETH-C2 to C32, ETH-C3 to C30, ETH-C4 to C34, ETH-R1 to R35, ETH-R2 to R34, ETH-R3 to R33, ETH-R6 to R30, ETH-R7 to R32, J1 to ANT2, JP_ESP_RX to JRX, JP_ESP_TX to JTX, PWR-SWT to PWR, RW5500-1 to R53, RW5500-2 to R52, RW5500-3 to R51, SIM900-C1 to C96, SIM900-C2 to C97, SIM900-LED1 to LED1, SIM900-LED2 to LED2, SIM900-R10 to R93, SIM900-R5 to R95, SIM900-R6 to R96, SIM900-R7 to R92, SIM900-R8 to R91, SIM900-R9 to R90, SIM900-T1 to T1, SIM900-T2 to T2, SIM900-T3 to T3, SIM_C1 to C80, SIM_C2 to C81, STM-C1 to C23, STM-C10 to C24, STM-C11 to C26, STM-C2 to C22, STM-C3 to C21, STM-C8 to C20, STM-L1 to L3, STM-XTAL to XTAL1, STM_CHIP to STMF401, SYS-C3 to C10, SYS-C4 to C11, SYS-L1 to L1, SYS-L2 to L2, SYS-R2 to R10, U$10 to TV16-2, U$11 to TV16-3, U$12 to TERM_BLOCK, U$13 to LCD14, U$14 to RJ-3, U$15 to RJ-2, U$16 to RJ-1, U$3 to HLK-PM01, U$5 to ESP, U$6 to DCDC, U$7 to ANT1, U$8 to SIMHOLDER, U$9 to TV16-1, W5500-C1 to C54, W5500-C10 to C51, W5500-C11 to C53, W5500-C12 to C37, W5500-C2 to C57, W5500-C3 to C52, W5500-C4 to C55, W5500-C5 to C56, W5500-C6 to C35, W5500-C7 to C33, W5500-C8 to C31, W5500-C9 to C50, W5500-R10 to R56, W5500-R11 to R50, W5500-R12 to R31, W5500-R13 to R54, W5500-XTAL to XTAL2
Connections:
- new net N$77: C28.1, STMF401.PB11
- net AGND: now also C25.2; no longer STM-C9.2
- net CC_GPIO0: now also STMF401.PH0_-OSC_IN; no longer STMF401.PH1-_OSC_OUT
- net DGND: now also C27.2, C28.2, LCD_C1.2; no longer STM-C12.2
- net MQ2_DATA: now also STMF401.PH1-_OSC_OUT; no longer STMF401.PB0
- net N$16: now also R94.1; no longer SIM900-R4.1
- net T_DO: now also STMF401.PB0; no longer STMF401.PB11
- net VCC: now also C25.1; no longer STM-C9.1
- net VDD: now also C27.1, LCD_C1.1, R94.2; no longer SIM900-R4.2, STM-C12.1
